Commit message: made all the files working

File: src/crn_robot_description/urdf/crn_robot_description.urdf (robot description, URDF)
Before this commit: robot pass Robot base chassis only, 5 links, 4 joints
Links:
- link base_link: geometry collision mesh filename=package://crn_robot_description/meshes/base_link.STL; visual mesh filename=package://crn_robot_description/meshes/base_link.STL
- link wheel_1: geometry collision mesh filename=package://crn_robot_description/meshes/wheel_1.STL; visual mesh filename=package://crn_robot_description/meshes/wheel_1.STL
- link wheel_2: geometry collision mesh filename=package://crn_robot_description/meshes/wheel_2.STL; visual mesh filename=package://crn_robot_description/meshes/wheel_2.STL
- link wheel_3: geometry collision mesh filename=package://crn_robot_description/meshes/wheel_3.STL; visual mesh filename=package://crn_robot_description/meshes/wheel_3.STL
- link wheel_4: geometry collision mesh filename=package://crn_robot_description/meshes/wheel_4.STL; visual mesh filename=package://crn_robot_description/meshes/wheel_4.STL
