Commit message: Made the following changes to urdf: Removed joint limits Changed joint type to continuous Increased velocity and effort limits Uncommented the trans file inclusion. Transmissions being used now Changed joint names by adding underscore
Changes to .gazebo file:
Commented skid steer drive. Only gazebo ros control plugin in use

Added config folder. Now the .rviz files can be used to load rviz configs

Added scripts folder to contain all nodes:
movement.py will contain the mechanics of movement of the bot.

Changes to joint_names.yaml:
Changed pid params

Changes to launch file:
Loaded controller information. Watch out for logs on terminal while launching
test.launch also launches rviz now. Sim starts off with pause off.

File: src/crn_robot_description/urdf/crn_robot_description.xacro (robot description, xacro)
@@ -6,5 +6,5 @@
   name="crn_robot_description" xmlns:xacro="http://www.ros.org/wiki/xacro">
 <xacro:include filename="$(find crn_robot_description)/urdf/crn_robot_description.gazebo" />
-<!--xacro:include filename="$(find crn_robot_description)/urdf/crn_robot_description.trans" /-->
+<xacro:include filename="$(find crn_robot_description)/urdf/crn_robot_description.trans" />
   <link
     name="base_link">
@@ -88,6 +88,6 @@
   </link>
   <joint
-    name="wheel_1"
-    type="revolute">
+    name="wheel_1_"
+    type="continuous">
     <origin
       xyz="0.30256 0.30135 0.023995"
@@ -98,10 +98,8 @@
       link="wheel_1" />
     <axis
-      xyz="1 0 -1" />
-    <limit
-      lower="0"
-      upper="1"
-      effort="0"
-      velocity="3" />
+      xyz="0 0 -1" />
+    <limit
+      effort="100"
+      velocity="50" />
   </joint>
   <link
@@ -146,6 +144,6 @@
   </link>
   <joint
-    name="wheel_2"
-    type="revolute">
+    name="wheel_2_"
+    type="continuous">
     <origin
       xyz="0.29811 -0.30581 0.024724"
@@ -156,10 +154,8 @@
       link="wheel_2" />
     <axis
-      xyz="1 0 1" />
-    <limit
-      lower="0"
-      upper="1"
-      effort="0"
-      velocity="3" />
+      xyz="0 0 1" />
+    <limit
+      effort="100"
+      velocity="50" />
   </joint>
   <link
@@ -204,6 +200,6 @@
   </link>
   <joint
-    name="wheel_3"
-    type="revolute">
+    name="wheel_3_"
+    type="continuous">
     <origin
       xyz="-0.29568 -0.30824 0.062368"
@@ -214,10 +210,8 @@
       link="wheel_3" />
     <axis
-      xyz="-1 0 1" />
-    <limit
-      lower="0"
-      upper="1"
-      effort="0"
-      velocity="3" />
+      xyz="0 0 1" />
+    <limit
+      effort="100"
+      velocity="50" />
   </joint>
   <link
@@ -262,6 +256,6 @@
   </link>
   <joint
-    name="wheel_4"
-    type="revolute">
+    name="wheel_4_"
+    type="continuous">
     <origin
       xyz="-0.31368 0.29024 0.05579"
@@ -272,10 +266,8 @@
       link="wheel_4" />
     <axis
-      xyz="-1 0 -1" />
-    <limit
-      lower="0"
-      upper="1"
-      effort="0"
-      velocity="3" />
+      xyz="0 0 -1" />
+    <limit
+      effort="100"
+      velocity="50" />
   </joint>
 </robot>
