Commit message: rack slider fixed

File: defense_bot_description/urdf/defense_bot.xacro (robot description, xacro)
@@ -6,4 +6,6 @@
 <xacro:include filename="$(find defense_bot_description)/gazebo/defense_bot_physics.gazebo" />
 <xacro:include filename="$(find defense_bot_description)/gazebo/defense_bot_plugins.gazebo" />
+<link name="dummy">
+</link>
 <link name="base_link">
   <inertial>
@@ -69,6 +71,6 @@
   <inertial>
     <origin rpy="0 0 0" xyz="0.009405 -0.117358 -0.381387"/>
-    <mass value="0.0"/>
-    <inertia ixx="0.0" ixy="0.0" ixz="0.0" iyy="0.0" iyz="0.0" izz="0.0"/>
+    <mass value="0.0001"/>
+    <inertia ixx="0.0001" ixy="0.0001" ixz="0.0001" iyy="0.0001" iyz="0.0001" izz="0.0001"/>
   </inertial>
   <visual>
@@ -118,5 +120,5 @@
     </geometry>
     <material name="silver_default"/>
-  </visual>
+    </visual>
   <collision>
     <origin rpy="0 0 0" xyz="-0.048894 -0.507834 -0.397687"/>
@@ -166,4 +168,8 @@
   </collision>
 </link>
+<joint name="dummy_joint" type="fixed">
+  <parent link="dummy"/>
+  <child link="base_link"/>
+</joint>
 <joint name="gripper_ball_rotation" type="continuous">
   <origin rpy="0 0 0" xyz="0.0 0.0 0.074203"/>

Commit message: URDF Fixed

File: defense_bot_description/urdf/defense_bot.xacro (robot description, xacro)
@@ -10,7 +10,7 @@
 <link name="base_link">
   <inertial>
-    <origin rpy="0 0 0" xyz="0.12099232848976177 0.12384344744617357 0.09244265027127854"/>
-    <mass value="116.038743583541"/>
-    <inertia ixx="5.021883" ixy="-0.105373" ixz="-0.817134" iyy="7.490255" iyz="-0.038364" izz="11.54731"/>
+    <origin rpy="0 0 0" xyz="0.16659672308956103 0.1220108917610289 0.09994102500540585"/>
+    <mass value="87.8762825405215"/>
+    <inertia ixx="3.13013" ixy="-0.162358" ixz="-0.752534" iyy="4.617725" iyz="-0.037475" izz="6.886069"/>
   </inertial>
   <visual>
@@ -30,10 +30,10 @@
 <link name="gripper_ball_1">
   <inertial>
-    <origin rpy="0 0 0" xyz="-6.11849846898771e-08 -3.6474196332680897e-07 0.044306464815765056"/>
+    <origin rpy="0 0 0" xyz="3.02552427000613e-07 -2.384254182974388e-10 0.044306596545721444"/>
     <mass value="0.47356245578988415"/>
     <inertia ixx="0.000485" ixy="-0.0" ixz="0.0" iyy="0.000485" iyz="-0.0" izz="0.000508"/>
   </inertial>
   <visual>
-    <origin rpy="0 0 0" xyz="-0.349673 -0.131302 -0.667744"/>
+    <origin rpy="0 0 0" xyz="-0.35585 -0.133057 -0.670731"/>
     <geometry>
       <mesh filename="package://defense_bot_description/meshes/gripper_ball_1.stl" scale="0.001 0.001 0.001"/>
@@ -42,5 +42,5 @@
   </visual>
   <collision>
-    <origin rpy="0 0 0" xyz="-0.349673 -0.131302 -0.667744"/>
+    <origin rpy="0 0 0" xyz="-0.35585 -0.133057 -0.670731"/>
     <geometry>
       <mesh filename="package://defense_bot_description/meshes/gripper_ball_1.stl" scale="0.001 0.001 0.001"/>
@@ -48,12 +48,112 @@
   </collision>
 </link>
+<link name="rack_1">
+  <inertial>
+    <origin rpy="0 0 0" xyz="0.009405 -0.117358 -0.400287"/>
+    <mass value="0.0001"/>
+    <inertia ixx="0.0001" ixy="0.0001" ixz="0.0001" iyy="0.0001" iyz="0.0001" izz="0.0001"/>
+  </inertial>
+  <visual>
+    <origin rpy="0 0 0" xyz="0.009405 -0.117358 -0.400287"/>
+    <geometry>
+      <mesh filename="package://defense_bot_description/meshes/rack_1.stl" scale="0.001 0.001 0.001"/>
+    </geometry>
+    <material name="silver_default"/>
+  </visual>
+  <collision>
+    <origin rpy="0 0 0" xyz="0.009405 -0.117358 -0.400287"/>
+    <geometry>
+      <mesh filename="package://defense_bot_description/meshes/rack_1.stl" scale="0.001 0.001 0.001"/>
+    </geometry>
+  </collision>
+</link>
+<link name="screw_turn_1">
+  <inertial>
+    <origin rpy="0 0 0" xyz="-0.0032110045585751618 0.037437890732595736 -0.10784422197706228"/>
+    <mass value="0.5399709461576145"/>
+    <inertia ixx="0.000829" ixy="7.1e-05" ixz="6.6e-05" iyy="0.000428" iyz="-0.000218" izz="0.000511"/>
+  </inertial>
+  <visual>
+    <origin rpy="0 0 0" xyz="-0.046317 -0.472245 -0.526187"/>
+    <geometry>
+      <mesh filename="package://defense_bot_description/meshes/screw_turn_1.stl" scale="0.001 0.001 0.001"/>
+    </geometry>
+    <material name="silver_default"/>
+  </visual>
+  <collision>
+    <origin rpy="0 0 0" xyz="-0.046317 -0.472245 -0.526187"/>
+    <geometry>
+      <mesh filename="package://defense_bot_description/meshes/screw_turn_1.stl" scale="0.001 0.001 0.001"/>
+    </geometry>
+  </collision>
+</link>
+<link name="right_finger_1">
+  <inertial>
+    <origin rpy="0 0 0" xyz="0.008043035510031701 0.032527162838390744 0.029999999999994087"/>
+    <mass value="0.1895264462202996"/>
+    <inertia ixx="0.00012" ixy="-1e-05" ixz="0.0" iyy="6.6e-05" iyz="0.0" izz="7.3e-05"/>
+  </inertial>
+  <visual>
+    <origin rpy="0 0 0" xyz="-0.048894 -0.507834 -0.416587"/>
+    <geometry>
+      <mesh filename="package://defense_bot_description/meshes/right_finger_1.stl" scale="0.001 0.001 0.001"/>
+    </geometry>
+    <material name="silver_default"/>
+  </visual>
+  <collision>
+    <origin rpy="0 0 0" xyz="-0.048894 -0.507834 -0.416587"/>
+    <geometry>
+      <mesh filename="package://defense_bot_description/meshes/right_finger_1.stl" scale="0.001 0.001 0.001"/>
+    </geometry>
+  </collision>
+</link>
+<link name="gripper_1">
+  <inertial>
+    <origin rpy="0 0 0" xyz="-5.6142082997978626e-05 -5.377771144704502e-06 0.01257026583797427"/>
+    <mass value="1.1544288999081391"/>
+    <inertia ixx="0.000982" ixy="0.0" ixz="3e-06" iyy="0.001008" iyz="-0.0" izz="0.000357"/>
+  </inertial>
+  <visual>
+    <origin rpy="0 0 0" xyz="-0.35585 -0.133057 -0.596528"/>
+    <geometry>
+      <mesh filename="package://defense_bot_description/meshes/gripper_1.stl" scale="0.001 0.001 0.001"/>
+    </geometry>
+    <material name="silver_default"/>
+  </visual>
+  <collision>
+    <origin rpy="0 0 0" xyz="-0.35585 -0.133057 -0.596528"/>
+    <geometry>
+      <mesh filename="package://defense_bot_description/meshes/gripper_1.stl" scale="0.001 0.001 0.001"/>
+    </geometry>
+  </collision>
+</link>
+<link name="gripper_arm_1">
+  <inertial>
+    <origin rpy="0 0 0" xyz="3.027907947705799e-07 6.38378239159465e-16 0.20248213586701128"/>
+    <mass value="38.912224485646085"/>
+    <inertia ixx="0.684471" ixy="0.0" ixz="0.0" iyy="0.667687" iyz="0.0" izz="0.084993"/>
+  </inertial>
+  <visual>
+    <origin rpy="0 0 0" xyz="-0.35585 -0.133057 -0.166042"/>
+    <geometry>
+      <mesh filename="package://defense_bot_description/meshes/gripper_arm_1.stl" scale="0.001 0.001 0.001"/>
+    </geometry>
+    <material name="silver_default"/>
+  </visual>
+  <collision>
+    <origin rpy="0 0 0" xyz="-0.35585 -0.133057 -0.166042"/>
+    <geometry>
+      <mesh filename="package://defense_bot_description/meshes/gripper_arm_1.stl" scale="0.001 0.001 0.001"/>
+    </geometry>
+  </collision>
+</link>
 <link name="turn_table_1">
   <inertial>
-    <origin rpy="0 0 0" xyz="-0.00625093492919542 0.23970404427172037 0.32294960634579334"/>
+    <origin rpy="0 0 0" xyz="-0.006250934929195633 0.23970404427172046 0.32294960634579006"/>
     <mass value="14.511620008028595"/>
     <inertia ixx="0.717239" ixy="0.019632" ixz="0.006421" iyy="0.171852" iyz="-0.171252" izz="0.598756"/>
   </inertial>
   <visual>
-    <origin rpy="0 0 0" xyz="0.0 0.175 -0.041387"/>
+    <origin rpy="0 0 0" xyz="0.0 0.175 -0.060287"/>
     <geometry>
       <mesh filename="package://defense_bot_description/meshes/turn_table_1.stl" scale="0.001 0.001 0.001"/>
@@ -62,5 +162,5 @@
   </visual>
   <collision>
-    <origin rpy="0 0 0" xyz="0.0 0.175 -0.041387"/>
+    <origin rpy="0 0 0" xyz="0.0 0.175 -0.060287"/>
     <geometry>
       <mesh filename="package://defense_bot_description/meshes/turn_table_1.stl" scale="0.001 0.001 0.001"/>
@@ -68,101 +168,81 @@
   </collision>
 </link>
-<link name="rack_1">
-  <inertial>
-    <origin rpy="0 0 0" xyz="0.009405 -0.117358 -0.381387"/>
-    <mass value="0.0001"/>
-    <inertia ixx="0.0001" ixy="0.0001" ixz="0.0001" iyy="0.0001" iyz="0.0001" izz="0.0001"/>
-  </inertial>
-  <visual>
-    <origin rpy="0 0 0" xyz="0.009405 -0.117358 -0.381387"/>
-    <geometry>
-      <mesh filename="package://defense_bot_description/meshes/rack_1.stl" scale="0.001 0.001 0.001"/>
-    </geometry>
-    <material name="silver_default"/>
-  </visual>
-  <collision>
-    <origin rpy="0 0 0" xyz="0.009405 -0.117358 -0.381387"/>
-    <geometry>
-      <mesh filename="package://defense_bot_description/meshes/rack_1.stl" scale="0.001 0.001 0.001"/>
-    </geometry>
-  </collision>
-</link>
-<link name="screw_turn_1">
-  <inertial>
-    <origin rpy="0 0 0" xyz="-0.0032110045585751618 0.037437890732595736 -0.10784422197705906"/>
-    <mass value="0.5399709461576145"/>
-    <inertia ixx="0.000829" ixy="7.1e-05" ixz="6.6e-05" iyy="0.000428" iyz="-0.000218" izz="0.000511"/>
-  </inertial>
-  <visual>
-    <origin rpy="0 0 0" xyz="-0.046317 -0.472245 -0.507287"/>
-    <geometry>
-      <mesh filename="package://defense_bot_description/meshes/screw_turn_1.stl" scale="0.001 0.001 0.001"/>
-    </geometry>
-    <material name="silver_default"/>
-  </visual>
-  <collision>
-    <origin rpy="0 0 0" xyz="-0.046317 -0.472245 -0.507287"/>
-    <geometry>
-      <mesh filename="package://defense_bot_description/meshes/screw_turn_1.stl" scale="0.001 0.001 0.001"/>
-    </geometry>
-  </collision>
-</link>
-<link name="right_finger_1">
-  <inertial>
-    <origin rpy="0 0 0" xyz="0.008043035510031916 0.03252716283839108 0.02999999999999725"/>
-    <mass value="0.1895264462202996"/>
-    <inertia ixx="0.00012" ixy="-1e-05" ixz="0.0" iyy="6.6e-05" iyz="-0.0" izz="7.3e-05"/>
-  </inertial>
-  <visual>
-    <origin rpy="0 0 0" xyz="-0.048894 -0.507834 -0.397687"/>
-    <geometry>
-      <mesh filename="package://defense_bot_description/meshes/right_finger_1.stl" scale="0.001 0.001 0.001"/>
-    </geometry>
-    <material name="silver_default"/>
-    </visual>
-  <collision>
-    <origin rpy="0 0 0" xyz="-0.048894 -0.507834 -0.397687"/>
-    <geometry>
-      <mesh filename="package://defense_bot_description/meshes/right_finger_1.stl" scale="0.001 0.001 0.001"/>
-    </geometry>
-  </collision>
-</link>
-<link name="gripper_arm_1">
-  <inertial>
-    <origin rpy="0 0 0" xyz="-6.094661719746597e-08 -3.6450353810280056e-07 0.20248200413705514"/>
-    <mass value="38.912224485646085"/>
-    <inertia ixx="0.684471" ixy="-0.0" ixz="0.0" iyy="0.667687" iyz="0.0" izz="0.084993"/>
-  </inertial>
-  <visual>
-    <origin rpy="0 0 0" xyz="-0.349673 -0.131302 -0.163055"/>
-    <geometry>
-      <mesh filename="package://defense_bot_description/meshes/gripper_arm_1.stl" scale="0.001 0.001 0.001"/>
-    </geometry>
-    <material name="silver_default"/>
-  </visual>
-  <collision>
-    <origin rpy="0 0 0" xyz="-0.349673 -0.131302 -0.163055"/>
-    <geometry>
-      <mesh filename="package://defense_bot_description/meshes/gripper_arm_1.stl" scale="0.001 0.001 0.001"/>
-    </geometry>
-  </collision>
-</link>
-<link name="gripper_1">
-  <inertial>
-    <origin rpy="0 0 0" xyz="-5.650582040972463e-05 -5.742274682640769e-06 0.012570134108018105"/>
-    <mass value="1.1544288999081391"/>
-    <inertia ixx="0.000982" ixy="0.0" ixz="3e-06" iyy="0.001008" iyz="-0.0" izz="0.000357"/>
-  </inertial>
-  <visual>
-    <origin rpy="0 0 0" xyz="-0.349673 -0.131302 -0.593541"/>
-    <geometry>
-      <mesh filename="package://defense_bot_description/meshes/gripper_1.stl" scale="0.001 0.001 0.001"/>
-    </geometry>
-    <material name="silver_default"/>
-  </visual>
-  <collision>
-    <origin rpy="0 0 0" xyz="-0.349673 -0.131302 -0.593541"/>
-    <geometry>
-      <mesh filename="package://defense_bot_description/meshes/gripper_1.stl" scale="0.001 0.001 0.001"/>
+<link name="wheel_fr_1">
+  <inertial>
+    <origin rpy="0 0 0" xyz="0.03016532251169568 -0.03012921280061831 4.6264918548977185e-06"/>
+    <mass value="7.4484852299099815"/>
+    <inertia ixx="0.021357" ixy="0.001481" ixz="1e-06" iyy="0.021306" iyz="-1e-06" izz="0.022811"/>
+  </inertial>
+  <visual>
+    <origin rpy="0 0 0" xyz="-0.198717 0.136246 -0.084387"/>
+    <geometry>
+      <mesh filename="package://defense_bot_description/meshes/wheel_fr_1.stl" scale="0.001 0.001 0.001"/>
+    </geometry>
+    <material name="silver_default"/>
+  </visual>
+  <collision>
+    <origin rpy="0 0 0" xyz="-0.198717 0.136246 -0.084387"/>
+    <geometry>
+      <mesh filename="package://defense_bot_description/meshes/wheel_fr_1.stl" scale="0.001 0.001 0.001"/>
+    </geometry>
+  </collision>
+</link>
+<link name="wheel_fl_1">
+  <inertial>
+    <origin rpy="0 0 0" xyz="0.030129212800609873 0.030164935880424182 4.6264918590194215e-06"/>
+    <mass value="7.4484852299099815"/>
+    <inertia ixx="0.021306" ixy="-0.001481" ixz="1e-06" iyy="0.021357" iyz="1e-06" izz="0.022811"/>
+  </inertial>
+  <visual>
+    <origin rpy="0 0 0" xyz="-0.244303 -0.356951 -0.084387"/>
+    <geometry>
+      <mesh filename="package://defense_bot_description/meshes/wheel_fl_1.stl" scale="0.001 0.001 0.001"/>
+    </geometry>
+    <material name="silver_default"/>
+  </visual>
+  <collision>
+    <origin rpy="0 0 0" xyz="-0.244303 -0.356951 -0.084387"/>
+    <geometry>
+      <mesh filename="package://defense_bot_description/meshes/wheel_fl_1.stl" scale="0.001 0.001 0.001"/>
+    </geometry>
+  </collision>
+</link>
+<link name="wheel_bl_1">
+  <inertial>
+    <origin rpy="0 0 0" xyz="-0.03012891435420334 0.03016562095811426 -4.626491794293419e-06"/>
+    <mass value="7.4484852299099815"/>
+    <inertia ixx="0.021306" ixy="0.001481" ixz="1e-06" iyy="0.021357" iyz="-1e-06" izz="0.022811"/>
+  </inertial>
+  <visual>
+    <origin rpy="0 0 0" xyz="0.193717 -0.40236 -0.084387"/>
+    <geometry>
+      <mesh filename="package://defense_bot_description/meshes/wheel_bl_1.stl" scale="0.001 0.001 0.001"/>
+    </geometry>
+    <material name="silver_default"/>
+  </visual>
+  <collision>
+    <origin rpy="0 0 0" xyz="0.193717 -0.40236 -0.084387"/>
+    <geometry>
+      <mesh filename="package://defense_bot_description/meshes/wheel_bl_1.stl" scale="0.001 0.001 0.001"/>
+    </geometry>
+  </collision>
+</link>
+<link name="wheel_br_1">
+  <inertial>
+    <origin rpy="0 0 0" xyz="-0.029458514176917305 -0.0294214209417418 -4.626491796277943e-06"/>
+    <mass value="7.4484852299099815"/>
+    <inertia ixx="0.021357" ixy="-0.001481" ixz="1e-06" iyy="0.021306" iyz="1e-06" izz="0.022811"/>
+  </inertial>
+  <visual>
+    <origin rpy="0 0 0" xyz="0.239303 0.090837 -0.084387"/>
+    <geometry>
+      <mesh filename="package://defense_bot_description/meshes/wheel_br_1.stl" scale="0.001 0.001 0.001"/>
+    </geometry>
+    <material name="silver_default"/>
+  </visual>
+  <collision>
+    <origin rpy="0 0 0" xyz="0.239303 0.090837 -0.084387"/>
+    <geometry>
+      <mesh filename="package://defense_bot_description/meshes/wheel_br_1.stl" scale="0.001 0.001 0.001"/>
     </geometry>
   </collision>
@@ -176,11 +256,5 @@
   <parent link="gripper_1"/>
   <child link="gripper_ball_1"/>
-  <axis xyz="-0.0 0.0 -1.0"/>
-</joint>
-<joint name="turn_table_rotation" type="continuous">
-  <origin rpy="0 0 0" xyz="0.0 -0.175 0.041387"/>
-  <parent link="base_link"/>
-  <child link="turn_table_1"/>
-  <axis xyz="0.0 -0.0 1.0"/>
+  <axis xyz="0.0 0.0 -1.0"/>
 </joint>
 <joint name="rack_slider" type="prismatic">
@@ -204,10 +278,4 @@
   <axis xyz="0.0 -0.0 1.0"/>
 </joint>
-<joint name="gripper_arm_rotation" type="continuous">
-  <origin rpy="0 0 0" xyz="0.349673 0.131302 0.163055"/>
-  <parent link="base_link"/>
-  <child link="gripper_arm_1"/>
-  <axis xyz="-0.0 1.0 0.0"/>
-</joint>
 <joint name="gripper_rotation" type="continuous">
   <origin rpy="0 0 0" xyz="0.0 0.0 0.430486"/>
@@ -216,3 +284,35 @@
   <axis xyz="-0.0 1.0 0.0"/>
 </joint>
+<joint name="gripper_arm_rotation" type="continuous">
+  <origin rpy="0 0 0" xyz="0.35585 0.133057 0.166042"/>
+  <parent link="base_link"/>
+  <child link="gripper_arm_1"/>
+  <axis xyz="0.0 -1.0 -0.0"/>
+</joint>
+<joint name="turn_table_rotation" type="continuous">
+  <origin rpy="0 0 0" xyz="0.0 -0.175 0.060287"/>
+  <parent link="base_link"/>
+  <child link="turn_table_1"/>
+  <axis xyz="0.0 -0.0 1.0"/>
+</joint>
+<joint name="wheel_fr_fix" type="fixed">
+  <origin rpy="0 0 0" xyz="0.198717 -0.136246 0.084387"/>
+  <parent link="base_link"/>
+  <child link="wheel_fr_1"/>
+</joint>
+<joint name="wheel_fl_fix" type="fixed">
+  <origin rpy="0 0 0" xyz="0.244303 0.356951 0.084387"/>
+  <parent link="base_link"/>
+  <child link="wheel_fl_1"/>
+</joint>
+<joint name="wheel_bl_fix" type="fixed">
+  <origin rpy="0 0 0" xyz="-0.193717 0.40236 0.084387"/>
+  <parent link="base_link"/>
+  <child link="wheel_bl_1"/>
+</joint>
+<joint name="wheel_br_fix" type="fixed">
+  <origin rpy="0 0 0" xyz="-0.239303 -0.090837 0.084387"/>
+  <parent link="base_link"/>
+  <child link="wheel_br_1"/>
+</joint>
 </robot>
