Commit message: gripper changes made

File: throwing_bot_description/urdf/throwing_bot.xacro (robot description, xacro)
@@ -10,7 +10,7 @@
 <link name="base_link">
   <inertial>
-    <origin rpy="0 0 0" xyz="-0.011851492296889534 -0.011348619168771903 0.25026581308769047"/>
-    <mass value="366.59500307051474"/>
-    <inertia ixx="42.733155" ixy="0.746789" ixz="0.016517" iyy="42.73439" iyz="0.005791" izz="68.525861"/>
+    <origin rpy="0 0 0" xyz="-0.011726915164729915 -0.011147209992249073 0.2397796079481494"/>
+    <mass value="317.96687849022385"/>
+    <inertia ixx="35.143458" ixy="0.812101" ixz="0.024376" iyy="35.144731" iyz="0.019118" izz="57.642285"/>
   </inertial>
   <visual>
@@ -30,10 +30,10 @@
 <link name="rotating_chamber_roller_fr_2_1">
   <inertial>
-    <origin rpy="0 0 0" xyz="9.510225135178629e-08 1.3912592169984528e-07 -0.00014705021665484264"/>
+    <origin rpy="0 0 0" xyz="9.51022514628086e-08 1.3912592186637873e-07 -0.00014705021665489815"/>
     <mass value="0.16224172662152384"/>
     <inertia ixx="4.6e-03" ixy="1.5e-03" ixz="0.0" iyy="4.6e-03" iyz="-0.0" izz="3.2e-03"/>
   </inertial>
   <visual>
-    <origin rpy="0 0 0" xyz="-0.278375 0.062874 -0.313183"/>
+    <origin rpy="0 0 0" xyz="-0.278375 0.062874 -0.273183"/>
     <geometry>
       <mesh filename="package://throwing_bot_description/meshes/rotating_chamber_roller_fr_2_1.stl" scale="0.001 0.001 0.001"/>
@@ -42,5 +42,5 @@
   </visual>
   <collision>
-    <origin rpy="0 0 0" xyz="-0.278375 0.062874 -0.313183"/>
+    <origin rpy="0 0 0" xyz="-0.278375 0.062874 -0.273183"/>
     <geometry>
       <mesh filename="package://throwing_bot_description/meshes/rotating_chamber_roller_fr_2_1.stl" scale="0.001 0.001 0.001"/>
@@ -50,10 +50,10 @@
 <link name="rotating_chamber_roller_fr_1_1">
   <inertial>
-    <origin rpy="0 0 0" xyz="-2.1050117549742398e-07 -1.664775036713806e-07 -0.0001470502166586729"/>
+    <origin rpy="0 0 0" xyz="-2.1050117539334057e-07 -1.6647750339382483e-07 -0.0001470502166586729"/>
     <mass value="0.16224172662152384"/>
     <inertia ixx="4.6e-03" ixy="1.5e-03" ixz="0.0" iyy="4.6e-03" iyz="-0.0" izz="3.2e-03"/>
   </inertial>
   <visual>
-    <origin rpy="0 0 0" xyz="-0.037959 0.30329 -0.313183"/>
+    <origin rpy="0 0 0" xyz="-0.037959 0.30329 -0.273183"/>
     <geometry>
       <mesh filename="package://throwing_bot_description/meshes/rotating_chamber_roller_fr_1_1.stl" scale="0.001 0.001 0.001"/>
@@ -62,5 +62,5 @@
   </visual>
   <collision>
-    <origin rpy="0 0 0" xyz="-0.037959 0.30329 -0.313183"/>
+    <origin rpy="0 0 0" xyz="-0.037959 0.30329 -0.273183"/>
     <geometry>
       <mesh filename="package://throwing_bot_description/meshes/rotating_chamber_roller_fr_1_1.stl" scale="0.001 0.001 0.001"/>
@@ -70,10 +70,10 @@
 <link name="rotating_chamber_roller_bl_1_1">
   <inertial>
-    <origin rpy="0 0 0" xyz="2.1607366701426045e-07 4.0694766339360866e-07 -0.0001470502166551202"/>
+    <origin rpy="0 0 0" xyz="2.1607366723630506e-07 4.069476635532032e-07 0.00014646283254493575"/>
     <mass value="0.16224172662152384"/>
     <inertia ixx="4.6e-03" ixy="1.5e-03" ixz="-0.0" iyy="4.6e-03" iyz="0.0" izz="3.2e-03"/>
   </inertial>
   <visual>
-    <origin rpy="0 0 0" xyz="0.306074 -0.040742 -0.313183"/>
+    <origin rpy="0 0 0" xyz="0.306074 -0.040742 -0.273183"/>
     <geometry>
       <mesh filename="package://throwing_bot_description/meshes/rotating_chamber_roller_bl_1_1.stl" scale="0.001 0.001 0.001"/>
@@ -82,5 +82,5 @@
   </visual>
   <collision>
-    <origin rpy="0 0 0" xyz="0.306074 -0.040742 -0.313183"/>
+    <origin rpy="0 0 0" xyz="0.306074 -0.040742 -0.273183"/>
     <geometry>
       <mesh filename="package://throwing_bot_description/meshes/rotating_chamber_roller_bl_1_1.stl" scale="0.001 0.001 0.001"/>
@@ -90,10 +90,10 @@
 <link name="rotating_chamber_roller_bl_2_1">
   <inertial>
-    <origin rpy="0 0 0" xyz="-4.783229013288759e-07 -2.874489165582972e-07 -0.0001470502166511789"/>
+    <origin rpy="0 0 0" xyz="-4.783229011345869e-07 -2.8744891639176373e-07 0.0001464628325491546"/>
     <mass value="0.16224172662152384"/>
     <inertia ixx="4.6e-03" ixy="1.5e-03" ixz="-0.0" iyy="4.6e-03" iyz="0.0" izz="3.2e-03"/>
   </inertial>
   <visual>
-    <origin rpy="0 0 0" xyz="0.065657 -0.281159 -0.313183"/>
+    <origin rpy="0 0 0" xyz="0.065657 -0.281159 -0.273183"/>
     <geometry>
       <mesh filename="package://throwing_bot_description/meshes/rotating_chamber_roller_bl_2_1.stl" scale="0.001 0.001 0.001"/>
@@ -102,5 +102,5 @@
   </visual>
   <collision>
-    <origin rpy="0 0 0" xyz="0.065657 -0.281159 -0.313183"/>
+    <origin rpy="0 0 0" xyz="0.065657 -0.281159 -0.273183"/>
     <geometry>
       <mesh filename="package://throwing_bot_description/meshes/rotating_chamber_roller_bl_2_1.stl" scale="0.001 0.001 0.001"/>
@@ -110,10 +110,10 @@
 <link name="gripper_arm_fr_1">
   <inertial>
-    <origin rpy="0 0 0" xyz="-1.3977562096645357e-07 4.770616842675324e-07 0.1619859252578661"/>
+    <origin rpy="0 0 0" xyz="-1.3977562079992012e-07 4.770616845450881e-07 0.16198592525786618"/>
     <mass value="19.9230589366508"/>
     <inertia ixx="0.221537" ixy="-0.00275" ixz="0.0" iyy="0.221537" iyz="0.0" izz="0.027851"/>
   </inertial>
   <visual>
-    <origin rpy="0 0 0" xyz="-0.333156 0.358242 -0.282924"/>
+    <origin rpy="0 0 0" xyz="-0.333156 0.358242 -0.242924"/>
     <geometry>
       <mesh filename="package://throwing_bot_description/meshes/gripper_arm_fr_1.stl" scale="0.001 0.001 0.001"/>
@@ -122,5 +122,5 @@
   </visual>
   <collision>
-    <origin rpy="0 0 0" xyz="-0.333156 0.358242 -0.282924"/>
+    <origin rpy="0 0 0" xyz="-0.333156 0.358242 -0.242924"/>
     <geometry>
       <mesh filename="package://throwing_bot_description/meshes/gripper_arm_fr_1.stl" scale="0.001 0.001 0.001"/>
@@ -130,10 +130,10 @@
 <link name="gripper_arm_bl_1">
   <inertial>
-    <origin rpy="0 0 0" xyz="4.959851587771347e-07 -1.5869908842613967e-07 0.16198592525786654"/>
+    <origin rpy="0 0 0" xyz="4.959851588326458e-07 -1.5869908820409506e-07 0.16198592525786656"/>
     <mass value="19.9230589366508"/>
     <inertia ixx="0.221537" ixy="-0.00275" ixz="0.0" iyy="0.221537" iyz="-0.0" izz="0.027851"/>
   </inertial>
   <visual>
-    <origin rpy="0 0 0" xyz="0.358242 -0.333156 -0.282924"/>
+    <origin rpy="0 0 0" xyz="0.358242 -0.333156 -0.242924"/>
     <geometry>
       <mesh filename="package://throwing_bot_description/meshes/gripper_arm_bl_1.stl" scale="0.001 0.001 0.001"/>
@@ -142,5 +142,5 @@
   </visual>
   <collision>
-    <origin rpy="0 0 0" xyz="0.358242 -0.333156 -0.282924"/>
+    <origin rpy="0 0 0" xyz="0.358242 -0.333156 -0.242924"/>
     <geometry>
       <mesh filename="package://throwing_bot_description/meshes/gripper_arm_bl_1.stl" scale="0.001 0.001 0.001"/>
@@ -150,10 +150,10 @@
 <link name="gripper_fr_1">
   <inertial>
-    <origin rpy="0 0 0" xyz="3.4946211526054594e-05 -2.8408082730801976e-05 0.010056153876451202"/>
+    <origin rpy="0 0 0" xyz="3.494621152599908e-05 -2.8408082730690953e-05 0.01005615387645109"/>
     <mass value="0.5910681632638519"/>
     <inertia ixx="0.000326" ixy="4e-02" ixz="-1e-02" iyy="0.000326" iyz="1e-02" izz="0.000117"/>
   </inertial>
   <visual>
-    <origin rpy="0 0 0" xyz="-0.333156 0.358242 -0.627313"/>
+    <origin rpy="0 0 0" xyz="-0.333156 0.358242 -0.587313"/>
     <geometry>
       <mesh filename="package://throwing_bot_description/meshes/gripper_fr_1.stl" scale="0.001 0.001 0.001"/>
@@ -162,5 +162,5 @@
   </visual>
   <collision>
-    <origin rpy="0 0 0" xyz="-0.333156 0.358242 -0.627313"/>
+    <origin rpy="0 0 0" xyz="-0.333156 0.358242 -0.587313"/>
     <geometry>
       <mesh filename="package://throwing_bot_description/meshes/gripper_fr_1.stl" scale="0.001 0.001 0.001"/>
@@ -170,10 +170,10 @@
 <link name="gripper_ball_fr_1">
   <inertial>
-    <origin rpy="0 0 0" xyz="-1.3950968558162913e-07 4.770693825539851e-07 0.035467027155031694"/>
+    <origin rpy="0 0 0" xyz="-1.3950968541509567e-07 4.770693827760297e-07 0.035467027155031805"/>
     <mass value="0.24291657027929903"/>
     <inertia ixx="0.000159" ixy="0.0" ixz="-0.0" iyy="0.000159" iyz="-0.0" izz="0.000167"/>
   </inertial>
   <visual>
-    <origin rpy="0 0 0" xyz="-0.333156 0.358242 -0.686676"/>
+    <origin rpy="0 0 0" xyz="-0.333156 0.358242 -0.646676"/>
     <geometry>
       <mesh filename="package://throwing_bot_description/meshes/gripper_ball_fr_1.stl" scale="0.001 0.001 0.001"/>
@@ -182,5 +182,5 @@
   </visual>
   <collision>
-    <origin rpy="0 0 0" xyz="-0.333156 0.358242 -0.686676"/>
+    <origin rpy="0 0 0" xyz="-0.333156 0.358242 -0.646676"/>
     <geometry>
       <mesh filename="package://throwing_bot_description/meshes/gripper_ball_fr_1.stl" scale="0.001 0.001 0.001"/>
@@ -190,10 +190,10 @@
 <link name="gripper_bl_1">
   <inertial>
-    <origin rpy="0 0 0" xyz="2.9381129570626996e-05 -3.52446862355027e-05 0.010056153876451646"/>
+    <origin rpy="0 0 0" xyz="2.938112957079353e-05 -3.524468623544719e-05 0.010056153876451757"/>
     <mass value="0.5910681632638507"/>
     <inertia ixx="0.000326" ixy="4e-02" ixz="-1e-02" iyy="0.000326" iyz="1e-02" izz="0.000117"/>
   </inertial>
   <visual>
-    <origin rpy="0 0 0" xyz="0.358242 -0.333156 -0.627313"/>
+    <origin rpy="0 0 0" xyz="0.358242 -0.333156 -0.587313"/>
     <geometry>
       <mesh filename="package://throwing_bot_description/meshes/gripper_bl_1.stl" scale="0.001 0.001 0.001"/>
@@ -202,5 +202,5 @@
   </visual>
   <collision>
-    <origin rpy="0 0 0" xyz="0.358242 -0.333156 -0.627313"/>
+    <origin rpy="0 0 0" xyz="0.358242 -0.333156 -0.587313"/>
     <geometry>
       <mesh filename="package://throwing_bot_description/meshes/gripper_bl_1.stl" scale="0.001 0.001 0.001"/>
@@ -210,10 +210,10 @@
 <link name="gripper_ball_bl_1">
   <inertial>
-    <origin rpy="0 0 0" xyz="4.959812163751742e-07 -1.5897285232657765e-07 0.03546702715932504"/>
+    <origin rpy="0 0 0" xyz="4.959812164306854e-07 -1.589728521600442e-07 0.03546702715932515"/>
     <mass value="0.24291657038309492"/>
     <inertia ixx="0.000159" ixy="0.0" ixz="0.0" iyy="0.000159" iyz="-0.0" izz="0.000167"/>
   </inertial>
   <visual>
-    <origin rpy="0 0 0" xyz="0.358242 -0.333156 -0.686676"/>
+    <origin rpy="0 0 0" xyz="0.358242 -0.333156 -0.646676"/>
     <geometry>
       <mesh filename="package://throwing_bot_description/meshes/gripper_ball_bl_1.stl" scale="0.001 0.001 0.001"/>
@@ -222,5 +222,5 @@
   </visual>
   <collision>
-    <origin rpy="0 0 0" xyz="0.358242 -0.333156 -0.686676"/>
+    <origin rpy="0 0 0" xyz="0.358242 -0.333156 -0.646676"/>
     <geometry>
       <mesh filename="package://throwing_bot_description/meshes/gripper_ball_bl_1.stl" scale="0.001 0.001 0.001"/>
@@ -230,10 +230,10 @@
 <link name="arrow_holder_1">
   <inertial>
-    <origin rpy="0 0 0" xyz="-0.0031007846752700574 -0.04280260134703126 0.012073902838845851"/>
+    <origin rpy="0 0 0" xyz="-0.0031012243650013482 -0.04280305996033454 0.012073902839088657"/>
     <mass value="0.5992891515771885"/>
     <inertia ixx="0.00072" ixy="0.000361" ixz="1.3e-02" iyy="0.000719" iyz="1.2e-02" izz="0.000914"/>
   </inertial>
   <visual>
-    <origin rpy="0 0 0" xyz="-0.147275 -0.189701 -0.325039"/>
+    <origin rpy="0 0 0" xyz="-0.149004 -0.19143 -0.285039"/>
     <geometry>
       <mesh filename="package://throwing_bot_description/meshes/arrow_holder_1.stl" scale="0.001 0.001 0.001"/>
@@ -242,5 +242,5 @@
   </visual>
   <collision>
-    <origin rpy="0 0 0" xyz="-0.147275 -0.189701 -0.325039"/>
+    <origin rpy="0 0 0" xyz="-0.149004 -0.19143 -0.285039"/>
     <geometry>
       <mesh filename="package://throwing_bot_description/meshes/arrow_holder_1.stl" scale="0.001 0.001 0.001"/>
@@ -250,10 +250,10 @@
 <link name="slider_rod_2">
   <inertial>
-    <origin rpy="0 0 0" xyz="-0.23568382593868098 -0.40627933785324843 0.030589993822034367"/>
+    <origin rpy="0 0 0" xyz="-0.23395526562850028 -0.40455079646653846 0.030589993822032202"/>
     <mass value="1.9072467651966203"/>
     <inertia ixx="0.007541" ixy="0.006722" ixz="1.4e-02" iyy="0.007536" iyz="3.3e-02" izz="0.013661"/>
   </inertial>
   <visual>
-    <origin rpy="0 0 0" xyz="0.096358 -0.073407 -0.263416"/>
+    <origin rpy="0 0 0" xyz="0.096358 -0.073407 -0.223416"/>
     <geometry>
       <mesh filename="package://throwing_bot_description/meshes/slider_rod_2.stl" scale="0.001 0.001 0.001"/>
@@ -262,5 +262,5 @@
   </visual>
   <collision>
-    <origin rpy="0 0 0" xyz="0.096358 -0.073407 -0.263416"/>
+    <origin rpy="0 0 0" xyz="0.096358 -0.073407 -0.223416"/>
     <geometry>
       <mesh filename="package://throwing_bot_description/meshes/slider_rod_2.stl" scale="0.001 0.001 0.001"/>
@@ -270,10 +270,10 @@
 <link name="throwing_base_1">
   <inertial>
-    <origin rpy="0 0 0" xyz="0.3573047240161689 0.3572198634283679 -0.000726381651222685"/>
+    <origin rpy="0 0 0" xyz="0.35730528432643766 0.3572204048150748 -0.0007263816510170717"/>
     <mass value="83.15108258777522"/>
     <inertia ixx="3.06197" ixy="-2.3335" ixz="-0.039769" iyy="3.062187" iyz="-0.039717" izz="6.037185"/>
   </inertial>
   <visual>
-    <origin rpy="0 0 0" xyz="0.332917 0.332917 -0.304376"/>
+    <origin rpy="0 0 0" xyz="0.331189 0.331189 -0.264376"/>
     <geometry>
       <mesh filename="package://throwing_bot_description/meshes/throwing_base_1.stl" scale="0.001 0.001 0.001"/>
@@ -282,5 +282,5 @@
   </visual>
   <collision>
-    <origin rpy="0 0 0" xyz="0.332917 0.332917 -0.304376"/>
+    <origin rpy="0 0 0" xyz="0.331189 0.331189 -0.264376"/>
     <geometry>
       <mesh filename="package://throwing_bot_description/meshes/throwing_base_1.stl" scale="0.001 0.001 0.001"/>
@@ -288,90 +288,170 @@
   </collision>
 </link>
-<link name="arrow_grasper_1_2">
-  <inertial>
-    <origin rpy="0 0 0" xyz="0.0019773748334052862 -0.002102348841381718 0.06444741353722411"/>
-    <mass value="0.2227546747031532"/>
-    <inertia ixx="0.000447" ixy="3e-02" ixz="-1.3e-02" iyy="0.000447" iyz="1.4e-02" izz="1e-02"/>
-  </inertial>
-  <visual>
-    <origin rpy="0 0 0" xyz="0.022332 0.217672 -0.304788"/>
-    <geometry>
-      <mesh filename="package://throwing_bot_description/meshes/arrow_grasper_1_2.stl" scale="0.001 0.001 0.001"/>
-    </geometry>
-    <material name="silver_default"/>
-  </visual>
-  <collision>
-    <origin rpy="0 0 0" xyz="0.022332 0.217672 -0.304788"/>
-    <geometry>
-      <mesh filename="package://throwing_bot_description/meshes/arrow_grasper_1_2.stl" scale="0.001 0.001 0.001"/>
-    </geometry>
-  </collision>
-</link>
-<link name="arrow_grasper_2_2">
-  <inertial>
-    <origin rpy="0 0 0" xyz="0.0019775570824419053 -0.0021021653508950765 0.0644466168155644"/>
-    <mass value="0.22275467470315166"/>
-    <inertia ixx="0.000447" ixy="3e-02" ixz="-1.3e-02" iyy="0.000447" iyz="1.4e-02" izz="1e-02"/>
-  </inertial>
-  <visual>
-    <origin rpy="0 0 0" xyz="-0.172122 0.023218 -0.305165"/>
-    <geometry>
-      <mesh filename="package://throwing_bot_description/meshes/arrow_grasper_2_2.stl" scale="0.001 0.001 0.001"/>
-    </geometry>
-    <material name="silver_default"/>
-  </visual>
-  <collision>
-    <origin rpy="0 0 0" xyz="-0.172122 0.023218 -0.305165"/>
-    <geometry>
-      <mesh filename="package://throwing_bot_description/meshes/arrow_grasper_2_2.stl" scale="0.001 0.001 0.001"/>
-    </geometry>
-  </collision>
-</link>
-<link name="arrow_grasper_4_2">
-  <inertial>
-    <origin rpy="0 0 0" xyz="-0.001977883687975787 0.0018532606170429955 0.06445426800904086"/>
-    <mass value="0.2227546747031517"/>
-    <inertia ixx="0.000447" ixy="3e-02" ixz="1.3e-02" iyy="0.000447" iyz="-1.2e-02" izz="1e-02"/>
-  </inertial>
-  <visual>
-    <origin rpy="0 0 0" xyz="0.022803 -0.171707 -0.305165"/>
-    <geometry>
-      <mesh filename="package://throwing_bot_description/meshes/arrow_grasper_4_2.stl" scale="0.001 0.001 0.001"/>
-    </geometry>
-    <material name="silver_default"/>
-  </visual>
-  <collision>
-    <origin rpy="0 0 0" xyz="0.022803 -0.171707 -0.305165"/>
-    <geometry>
-      <mesh filename="package://throwing_bot_description/meshes/arrow_grasper_4_2.stl" scale="0.001 0.001 0.001"/>
-    </geometry>
-  </collision>
-</link>
-<link name="arrow_grasper_3_2">
-  <inertial>
-    <origin rpy="0 0 0" xyz="-0.0019770671784639926 0.0018530783680034517 0.06445506473310253"/>
-    <mass value="0.2227546747031532"/>
-    <inertia ixx="0.000447" ixy="3e-02" ixz="1.3e-02" iyy="0.000447" iyz="-1.2e-02" izz="1e-02"/>
-  </inertial>
-  <visual>
-    <origin rpy="0 0 0" xyz="0.217258 0.022747 -0.304788"/>
-    <geometry>
-      <mesh filename="package://throwing_bot_description/meshes/arrow_grasper_3_2.stl" scale="0.001 0.001 0.001"/>
-    </geometry>
-    <material name="silver_default"/>
-  </visual>
-  <collision>
-    <origin rpy="0 0 0" xyz="0.217258 0.022747 -0.304788"/>
-    <geometry>
-      <mesh filename="package://throwing_bot_description/meshes/arrow_grasper_3_2.stl" scale="0.001 0.001 0.001"/>
-    </geometry>
-  </collision>
-</link>
-<joint name="dummy_joint" type="fixed">
+<link name="wheel_fl_1">
+  <inertial>
+    <origin rpy="0 0 0" xyz="0.031542608490837065 -0.03157966654337491 -4.62912066842569e-06"/>
+    <mass value="7.448486590236144"/>
+    <inertia ixx="0.021306" ixy="0.001481" ixz="-1e-06" iyy="0.021358" iyz="1e-06" izz="0.022811"/>
+  </inertial>
+  <visual>
+    <origin rpy="0 0 0" xyz="-0.261415 0.2865 -0.0819"/>
+    <geometry>
+      <mesh filename="package://throwing_bot_description/meshes/wheel_fl_1.stl" scale="0.001 0.001 0.001"/>
+    </geometry>
+    <material name="silver_default"/>
+  </visual>
+  <collision>
+    <origin rpy="0 0 0" xyz="-0.261415 0.2865 -0.0819"/>
+    <geometry>
+      <mesh filename="package://throwing_bot_description/meshes/wheel_fl_1.stl" scale="0.001 0.001 0.001"/>
+    </geometry>
+  </collision>
+</link>
+<link name="wheel_br_1">
+  <inertial>
+    <origin rpy="0 0 0" xyz="-0.030165434057531304 -0.030129057642393764 -4.629120670326947e-06"/>
+    <mass value="7.448486590236144"/>
+    <inertia ixx="0.021358" ixy="-0.001481" ixz="1e-06" iyy="0.021306" iyz="1e-06" izz="0.022811"/>
+  </inertial>
+  <visual>
+    <origin rpy="0 0 0" xyz="0.2865 0.2865 -0.0819"/>
+    <geometry>
+      <mesh filename="package://throwing_bot_description/meshes/wheel_br_1.stl" scale="0.001 0.001 0.001"/>
+    </geometry>
+    <material name="silver_default"/>
+  </visual>
+  <collision>
+    <origin rpy="0 0 0" xyz="0.2865 0.2865 -0.0819"/>
+    <geometry>
+      <mesh filename="package://throwing_bot_description/meshes/wheel_br_1.stl" scale="0.001 0.001 0.001"/>
+    </geometry>
+  </collision>
+</link>
+<link name="wheel_fr_1">
+  <inertial>
+    <origin rpy="0 0 0" xyz="0.028714181366090774 -0.02875123941862845 -4.629120668495079e-06"/>
+    <mass value="7.448486590236144"/>
+    <inertia ixx="0.021306" ixy="0.001481" ixz="-1e-06" iyy="0.021358" iyz="1e-06" izz="0.022811"/>
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